Commit message: Update BPX robot model assets

File: bpx/urdf/bpx.urdf (robot description, URDF)
Before this commit: robot bpx, 17 links, 16 joints
Links:
- link fl_calf_link: mass 0.294 -> 0.253; geometry collision box size=0.02 0.02 0.15; collision box size=0.03 0.02 0.07
- link fl_hip_link: mass 0.588 -> 0.554
- link fl_thigh_link: mass 1.74 -> 1.213; geometry collision box size=0.045 0.13 0.029; collision cylinder length=0.08 radius=0.044
- link fl_toe_link: mass 0.005 -> 0.062; geometry collision cylinder length=0.0358 radius=0.027; visual mesh filename=../meshes/toe.obj
- link fr_calf_link: mass 0.294 -> 0.253; geometry collision box size=0.02 0.02 0.15; collision box size=0.03 0.02 0.07
- link fr_hip_link: mass 0.588 -> 0.554
- link fr_thigh_link: mass 1.74 -> 1.213; geometry collision box size=0.045 0.13 0.029; collision cylinder length=0.08 radius=0.044
- link fr_toe_link: mass 0.005 -> 0.062; geometry collision cylinder length=0.0358 radius=0.027; visual mesh filename=../meshes/toe.obj
- link hl_calf_link: mass 0.294 -> 0.253; geometry collision box size=0.02 0.02 0.15; collision box size=0.03 0.02 0.07
- link hl_hip_link: mass 0.588 -> 0.554
- link hl_thigh_link: mass 1.74 -> 1.213; geometry collision box size=0.045 0.13 0.029; collision cylinder length=0.08 radius=0.044
- link hl_toe_link: mass 0.005 -> 0.062; geometry collision cylinder length=0.0358 radius=0.027; visual mesh filename=../meshes/toe.obj
- link hr_calf_link: mass 0.294 -> 0.253; geometry collision box size=0.02 0.02 0.15; collision box size=0.03 0.02 0.07
- link hr_hip_link: mass 0.588 -> 0.554
- link hr_thigh_link: mass 1.74 -> 1.213; geometry collision box size=0.045 0.13 0.029; collision cylinder length=0.08 radius=0.044
- link hr_toe_link: mass 0.005 -> 0.062; geometry collision cylinder length=0.0358 radius=0.027; visual mesh filename=../meshes/toe.obj
- link torso: mass 3.309 -> 6.829; geometry collision box size=0.01329 0.136 0.026; collision box size=0.01329 0.136 0.026
Joints:
- joint fl_ankle_joint: origin xyz=0 0 -0.2427 rpy=0 0 0 -> xyz=0 0 -0.2315648 rpy=0 0 0
- joint fl_hip_pitch_joint: limit lower=-0.7854 upper=2.6066 effort=30 velocity=20 -> lower=-0.7854 upper=2.60661 effort=30 velocity=20; origin xyz=0 0.1089 0 rpy=0 0 0 -> xyz=0 0.11522 0 rpy=0 0 0
- joint fl_hip_roll_joint: origin xyz=0.2432 0.056 0 rpy=0 0 0 -> xyz=0.2386 0.056 0 rpy=0 0 0
- joint fr_ankle_joint: origin xyz=0 0 -0.2427 rpy=0 0 0 -> xyz=0 0 -0.2315648 rpy=0 0 0
- joint fr_hip_pitch_joint: limit lower=-0.7854 upper=2.6066 effort=30 velocity=20 -> lower=-0.7854 upper=2.60661 effort=30 velocity=20; origin xyz=0 -0.1089 0 rpy=0 0 0 -> xyz=0 -0.11522 0 rpy=0 0 0
- joint fr_hip_roll_joint: origin xyz=0.2432 -0.056 0 rpy=0 0 0 -> xyz=0.2386 -0.056 0 rpy=0 0 0
- joint hl_ankle_joint: origin xyz=0 0 -0.2427 rpy=0 0 0 -> xyz=0 0 -0.2315648 rpy=0 0 0
- joint hl_hip_pitch_joint: limit lower=-0.7854 upper=2.6066 effort=30 velocity=20 -> lower=-0.7854 upper=2.60661 effort=30 velocity=20; origin xyz=0 0.1089 0 rpy=0 0 0 -> xyz=0 0.11522 0 rpy=0 0 0
- joint hl_hip_roll_joint: origin xyz=-0.2432 0.056 0 rpy=0 0 0 -> xyz=-0.2386 0.056 0 rpy=0 0 0
- joint hr_ankle_joint: origin xyz=0 0 -0.2427 rpy=0 0 0 -> xyz=0 0 -0.2315648 rpy=0 0 0
- joint hr_hip_pitch_joint: limit lower=-0.7854 upper=2.6066 effort=30 velocity=20 -> lower=-0.7854 upper=2.60661 effort=30 velocity=20; origin xyz=0 -0.1089 0 rpy=0 0 0 -> xyz=0 -0.11522 0 rpy=0 0 0
- joint hr_hip_roll_joint: origin xyz=-0.2432 -0.056 0 rpy=0 0 0 -> xyz=-0.2386 -0.056 0 rpy=0 0 0
